File: pcb/hw-tester.sch (KiCad schematic (older format))
At the start: 40 parts, among them J1 Port_A, J10 Connector, J11 UserLED, J12 SW_Pls, J13 SW_Min, J14 GND, J15 5V, J2 Port_B, J3 Port_C, J4 Port_D, J5 I2C, J6 AVR-ISP-6, J7 I2C, J8 Address, J9 Connector, K1 KEYSW, K2 KEYSW, SW1 SW_RESET, U1 ATmega32A-PU, U2 MCP23017_SP, Y1 Crystal

Commit message: Release v0.1
Parts:
- removed D3: D, symbol Device:D
- removed J2: Port_B, symbol Connector:Conn_01x05_Male
- removed J3: Port_C, symbol Connector:Conn_01x06_Male
- removed J5: I2C, symbol Connector:Conn_01x02_Male
- added J2: PORT_B, Connector_PinHeader_2.54mm:PinHeader_1x08_P2.54mm_Vertical, symbol Connector:Conn_01x08_Male
- added J3: PORT_C, Connector_PinHeader_2.54mm:PinHeader_1x08_P2.54mm_Vertical, symbol Connector:Conn_01x08_Male
- added JUSB1: USB_B, Connector_USB:USB_B_OST_USB-B1HSxx_Horizontal, symbol Connector:USB_B
- added SW2: SW_BOOT, Button_Switch_THT:SW_PUSH_6mm, symbol Switch:SW_Push
- C1, C2: value C -> 22p; footprint (none) -> Capacitor_THT:C_Disc_D3.8mm_W2.6mm_P2.50mm
- C3: footprint (none) -> Capacitor_THT:CP_Radial_D4.0mm_P1.50mm
- C4, C5: footprint (none) -> Capacitor_THT:C_Disc_D3.8mm_W2.6mm_P2.50mm
- D1, D2: footprint (none) -> Diode_THT:D_DO-35_SOD27_P7.62mm_Horizontal
- DL1, DL2, DL3: footprint (none) -> LED_THT:LED_D3.0mm
- F1: footprint (none) -> Capacitor_THT:C_Disc_D9.0mm_W5.0mm_P10.00mm
- J1: value Port_A -> PORT_A; footprint (none) -> Connector_PinHeader_2.54mm:PinHeader_1x08_P2.54mm_Vertical
- J10: value Connector -> PORT_GB; footprint (none) -> Connector_PinHeader_2.54mm:PinHeader_1x08_P2.54mm_Vertical
- J11, J12, J13, J7: footprint (none) -> Connector_PinHeader_2.54mm:PinHeader_1x02_P2.54mm_Vertical
- J4: value Port_D -> PORT_D; footprint (none) -> Connector_PinHeader_2.54mm:PinHeader_1x08_P2.54mm_Vertical
- J6: footprint (none) -> Connector_PinHeader_2.54mm:PinHeader_2x03_P2.54mm_Vertical
- J8: footprint (none) -> Connector_PinHeader_2.54mm:PinHeader_1x03_P2.54mm_Vertical
- J9: value Connector -> PORT_GA; footprint (none) -> Connector_PinHeader_2.54mm:PinHeader_1x08_P2.54mm_Vertical
- JG1: renamed from J14; footprint (none) -> Connector_PinHeader_2.54mm:PinHeader_1x05_P2.54mm_Vertical
- JV1: renamed from J15; footprint (none) -> Connector_PinHeader_2.54mm:PinHeader_1x05_P2.54mm_Vertical
- K1, K2: footprint (none) -> keebs:Mx_Alps_100
- PJ1: footprint (none) -> Connector_BarrelJack:BarrelJack_Horizontal
- R1: value R -> 10k; footprint (none) -> Resistor_THT:R_Axial_DIN0207_L6.3mm_D2.5mm_P7.62mm_Horizontal
- R2, R3: footprint (none) -> Resistor_THT:R_Axial_DIN0207_L6.3mm_D2.5mm_P7.62mm_Horizontal
- R4, R5, R6: renamed from R?; footprint (none) -> Resistor_THT:R_Axial_DIN0207_L6.3mm_D2.5mm_P7.62mm_Horizontal
- SW1: footprint (none) -> Button_Switch_THT:SW_PUSH_6mm
- U1: footprint Package_DIP:DIP-40_W15.24mm -> Package_DIP:DIP-40_W15.24mm_Socket
- U2: footprint Package_DIP:DIP-28_W7.62mm -> Package_DIP:DIP-28_W7.62mm_Socket
- Y1: footprint (none) -> Crystal:Crystal_HC49-U_Vertical
Connections:
- net +5V: now also JUSB1.1 (VBUS)
- net GND: now also JUSB1.4 (GND), JUSB1.5 (Shield), SW2.1
- net MISO: now also J2.7 (Pin_7)
- net MOSI: now also J2.6 (Pin_6)
- net SCK: now also J2.8 (Pin_8)
- net SCL: now also J3.1 (Pin_1)
- net SDA: now also J3.2 (Pin_2)
- net VCC: now also F1.2
- net PB0: now reaches U1.1 (PB0)
- net PB0: now also J2.1 (Pin_1)
- net PD0: now reaches J4.1 (Pin_1), U1.14 (PD0)
- net PD1: now reaches J4.2 (Pin_2), U1.15 (PD1)
- net D+: now reaches J4.3 (Pin_3), U1.16 (PD2)
- net D+: now also JUSB1.3 (D+)
- net D-: now reaches J4.4 (Pin_4), U1.17 (PD3)
- net D-: now also JUSB1.2 (D-)
- net BOOT: now reaches J4.5 (Pin_5), U1.18 (PD4)
- net BOOT: now also SW2.2
- net PD5: now reaches J4.6 (Pin_6), U1.19 (PD5)
- net PB1: now reaches U1.2 (PB1)
- net PB1: now also J2.2 (Pin_2)
- net PD6: now reaches J4.7 (Pin_7), U1.20 (PD6)
- net PD7: now reaches J4.8 (Pin_8), U1.21 (PD7)
- net PC2: now reaches U1.24 (PC2)
- net PC2: now also J3.3 (Pin_3)
- net PC3: now reaches U1.25 (PC3)
- net PC3: now also J3.4 (Pin_4)
- net PC4: now reaches U1.26 (PC4)
- net PC4: now also J3.5 (Pin_5)
- net PC5: now reaches U1.27 (PC5)
- net PC5: now also J3.6 (Pin_6)
- net PC6: now reaches U1.28 (PC6)
- net PC6: now also J3.7 (Pin_7)
- net PC7: now reaches U1.29 (PC7)
- net PC7: now also J3.8 (Pin_8)
- net PB2: now reaches U1.3 (PB2)
- net PB2: now also J2.3 (Pin_3)
- net PA7: now reaches J1.8 (Pin_8), U1.33 (PA7)
- net PA6: now reaches J1.7 (Pin_7), U1.34 (PA6)
- net PA5: now reaches J1.6 (Pin_6), U1.35 (PA5)
- net PA4: now reaches J1.5 (Pin_5), U1.36 (PA4)
- net PA3: now reaches J1.4 (Pin_4), U1.37 (PA3)
- net PA2: now reaches J1.3 (Pin_3), U1.38 (PA2)
- net PA1: now reaches J1.2 (Pin_2), U1.39 (PA1)
- net PB3: now reaches U1.4 (PB3)
- net PB3: now also J2.4 (Pin_4)
- net PA0: now reaches J1.1 (Pin_1), U1.40 (PA0)
- net PB4: now reaches U1.5 (PB4)
- net PB4: now also J2.5 (Pin_5)
- net GPA0: now reaches J9.1 (Pin_1)
- net GPA0: now also U2.21 (GPA0); no longer U2.1 (GPB0)
- net at U2.12 (SCK): now also J7.1 (Pin_1); no longer J7.2 (Pin_2)
- net at U2.13 (SDA): now also J7.2 (Pin_2); no longer J7.1 (Pin_1)
- net GPA1: now reaches J9.2 (Pin_2)
- net GPA1: now also U2.22 (GPA1); no longer U2.2 (GPB1)
- net GPB0: now reaches J10.1 (Pin_1)
- net GPB0: now also U2.1 (GPB0); no longer U2.21 (GPA0)
- net GPB1: now reaches J10.2 (Pin_2)
- net GPB1: now also U2.2 (GPB1); no longer U2.22 (GPA1)
- net GPA2: now reaches U2.23 (GPA2)
- net GPA2: now also J9.3 (Pin_3); no longer J10.3 (Pin_3)
- net GPA3: now reaches U2.24 (GPA3)
- net GPA3: now also J9.4 (Pin_4); no longer J10.4 (Pin_4)
- net GPA4: now reaches U2.25 (GPA4)
- net GPA4: now also J9.5 (Pin_5); no longer J10.5 (Pin_5)
- net GPA5: now reaches U2.26 (GPA5)
- net GPA5: now also J9.6 (Pin_6); no longer J10.6 (Pin_6)
- net GPA6: now reaches U2.27 (GPA6)
- net GPA6: now also J9.7 (Pin_7); no longer J10.7 (Pin_7)
- net GPA7: now reaches U2.28 (GPA7)
- net GPA7: now also J9.8 (Pin_8); no longer J10.8 (Pin_8)
- net GPB2: now reaches U2.3 (GPB2)
- net GPB2: now also J10.3 (Pin_3); no longer J9.3 (Pin_3)
- net GPB3: now reaches U2.4 (GPB3)
- net GPB3: now also J10.4 (Pin_4); no longer J9.4 (Pin_4)
- net GPB4: now reaches U2.5 (GPB4)
- net GPB4: now also J10.5 (Pin_5); no longer J9.5 (Pin_5)
- net GPB5: now reaches U2.6 (GPB5)
- net GPB5: now also J10.6 (Pin_6); no longer J9.6 (Pin_6)
- net GPB6: now reaches U2.7 (GPB6)
- net GPB6: now also J10.7 (Pin_7); no longer J9.7 (Pin_7)
- net GPB7: now reaches U2.8 (GPB7)
- net GPB7: now also J10.8 (Pin_8); no longer J9.8 (Pin_8)
Other:
- moved on the sheet: C3, C4, C5, DL1, DL2, DL3, F1, J10, J11, J6, J9, JG1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
